Commit message: Commit gustavo readme + gazebo

File: project_description/urdf/robutler.gazebo.xacro (robot description, xacro)
@@ -204,3 +204,15 @@
     </sensor>
   </gazebo>
+  <!-- Matro -->
+  <gazebo reference="mastro_link">
+    <material>Gazebo/Black</material>
+  </gazebo>
+  <!-- Antena -->
+  <gazebo reference="antena_link">
+    <material>Gazebo/Red</material>
+  </gazebo>
+    <!-- Castelo -->
+  <gazebo reference="castle_link">
+    <material>Gazebo/Blue</material>
+  </gazebo>
 </robot>

Commit message: commit câmera Gustavo

File: project_description/urdf/robutler.gazebo.xacro (robot description, xacro)
@@ -204,4 +204,38 @@
     </sensor>
   </gazebo>
+  <!-- Câmera Alta -->
+  <gazebo reference="camera_rgb_frame_alta">
+    <sensor type="camera" name="Pi Camera">
+      <always_on>true</always_on>
+      <visualize>$(arg camera_visual)</visualize>
+      <camera>
+          <horizontal_fov>1.085595</horizontal_fov>
+          <!-- <horizontal_fov>2.085595</horizontal_fov> -->
+          <image>
+              <width>640</width>
+              <height>480</height>
+              <format>R8G8B8</format>
+          </image>
+          <clip>
+              <near>0.03</near>
+              <far>100</far>
+          </clip>
+      </camera>
+      <plugin name="camera_controller_alta" filename="libgazebo_ros_camera.so">
+        <alwaysOn>true</alwaysOn>
+        <updateRate>30.0</updateRate>
+        <cameraName>camera</cameraName>
+        <frameName>camera_rgb_optical_frame_alta</frameName>
+        <imageTopicName>rgb/image_raw_up</imageTopicName>
+        <cameraInfoTopicName>rgb/camera_info_up</cameraInfoTopicName>
+        <hackBaseline>0.07</hackBaseline>
+        <distortionK1>0.0</distortionK1>
+        <distortionK2>0.0</distortionK2>
+        <distortionK3>0.0</distortionK3>
+        <distortionT1>0.0</distortionT1>
+        <distortionT2>0.0</distortionT2>
+      </plugin>
+    </sensor>
+  </gazebo>
   <!-- Matro -->
   <gazebo reference="mastro_link">

File: project_description/urdf/robutler.urdf.xacro (robot description, xacro)
@@ -213,4 +213,30 @@
   </joint>
   <link name="camera_rgb_optical_back"/>
+  <!-- Câmera Alta -->
+  <joint name="camera_joint_alta" type="fixed">
+    <origin xyz="0.073 -0.011 0.084" rpy="0 0 0"/>
+    <parent link="base_link"/>
+    <child link="camera_link_alta"/>
+  </joint>
+  <link name="camera_link_alta">
+    <collision>
+      <origin xyz="0.005 0.011 0.013" rpy="0 0 0"/>
+      <geometry>
+        <box size="0.015 0.030 0.027"/>
+      </geometry>
+    </collision>
+  </link>
+  <joint name="camera_rgb_joint_alta" type="fixed">
+    <origin xyz="0.003 0.011 2.009" rpy="0 0.35 0"/>
+    <parent link="camera_link_alta"/>
+    <child link="camera_rgb_frame_alta"/>
+  </joint>
+  <link name="camera_rgb_frame_alta"/>
+  <joint name="camera_rgb_optical_joint_alta" type="fixed">
+    <origin xyz="0 0 0" rpy="-1.57 0 -1.57"/>
+    <parent link="camera_rgb_frame_alta"/>
+    <child link="camera_rgb_optical_frame_alta"/>
+  </joint>
+  <link name="camera_rgb_optical_frame_alta"/>
   <!-- Estético adicional -->
   <!-- <joint name="antena" type="fixed">
