Commit message: commit meshes gustavo

File: project_description/urdf/robutler.urdf.xacro (robot description, xacro)
@@ -264,5 +264,5 @@
       <origin xyz="0 0 0.0" rpy="0 0 0"/>
       <geometry>
-        <mesh filename="package://turtlebot3_description/meshes/new/Pirate_Flag.stl" scale="0.002 0.002 0.002"/>
+        <mesh filename="package://project_description/meshes/new/Pirate_Flag.stl" scale="0.002 0.002 0.002"/>
       </geometry>
       <material name="red"/>
@@ -292,5 +292,5 @@
       <origin xyz="0 0 0.0" rpy="0 0 0"/>
       <geometry>
-        <mesh filename="package://turtlebot3_description/meshes/new/flag_cap.stl" scale="0.002 0.002 0.002"/>
+        <mesh filename="package://project_description/meshes/new/flag_cap.stl" scale="0.002 0.002 0.002"/>
       </geometry>
       <material name="red"/>

Commit message: commit Gustavo

File: project_description/urdf/robutler.urdf.xacro (robot description, xacro)
@@ -228,5 +228,5 @@
   </link>
   <joint name="camera_rgb_joint_alta" type="fixed">
-    <origin xyz="0.003 0.011 2.009" rpy="0 0.35 0"/>
+    <origin xyz="0.003 0.011 1.009" rpy="0 0.35 0"/>
     <parent link="camera_link_alta"/>
     <child link="camera_rgb_frame_alta"/>
